File: pcb_main/3340VCO_pcb_main.sch (KiCad schematic (older format))
At the start: 77 parts, among them J1 MJ-352, J2 MJ-352, J3 MJ-352, J4 POWER_IN, J5 MJ-352, J6 MJ-352, J7 MJ-352, U1 NJM074, U2 NJM074, U3 V3340M

Commit message: replace reference Diode: 1N5231B to LM336Z-5.0, update schematic and pcb
Parts:
- removed C7, C9: 2.2μ, Capacitor_THT:C_Disc_D5.1mm_W3.2mm_P5.00mm, symbol Device:C
- removed D2, D3: 1N5231B, Diode_THT:D_DO-34_SOD68_P7.62mm_Horizontal, symbol Device:D_Zener
- added D1, D2: LM336Z-5.0, Package_TO_SOT_THT:TO-92_Inline_Wide, symbol LM336:LM336
- added J8: EXT_POW, Connector_PinHeader_2.54mm:PinHeader_1x03_P2.54mm_Vertical, symbol Connector_Generic:Conn_01x03
- added TP1: VLFI, Connector_PinHeader_2.54mm:PinHeader_1x01_P2.54mm_Vertical, symbol Connector:TestPoint
- added TP2: VSSI, Connector_PinHeader_2.54mm:PinHeader_1x01_P2.54mm_Vertical, symbol Connector:TestPoint
- added TP3: VTO, Connector_PinHeader_2.54mm:PinHeader_1x01_P2.54mm_Vertical, symbol Connector:TestPoint
- added TP4: TRIOUT, Connector_PinHeader_2.54mm:PinHeader_1x01_P2.54mm_Vertical, symbol Connector:TestPoint
- C4: value 10n -> 0.1μ; footprint C_addition:C_Rect_L4.0mm_W2.5mm_P2.50mm -> Capacitor_THT:C_Rect_L7.2mm_W5.5mm_P5.00mm_FKS2_FKP2_MKS2_MKP2
- R23, R26: value 680 -> 1k
Connections:
- net +12V: now also J8.3 (Pin_3)
- net +5V: now also D1.2 (K)
- net -12V: now also J8.2 (Pin_2)
- net -5V: now also D2.3 (A)
- net GND: now also D1.3 (A), D2.2 (K), J8.1 (Pin_1)
- net at R29.2, U3.10 (VTO): now also TP3.1
- net at R18.2, R19.1, U3.13 (VLFI): now also TP1.1
- net at C4.1, U3.9 (VSSI): now also TP2.1
- net at J7.T, R41.1: now also TP4.1
- no-connect marks 12 -> 14
Changed lines of the file:
@@
 Wire Wire Line
 	7600 5750 7600 6850
-Wire Wire Line
-	8000 5950 8000 6850
-$Comp
-L Device:C C4
-U 1 1 5E86C6E8
-P 8000 7000
-F 0 "C4" H 8115 7046 50  0000 L CNN
-F 1 "10n" H 8115 6955 50  0000 L CNN
-F 2 "C_addition:C_Rect_L4.0mm_W2.5mm_P2.50mm" H 8038 6850 50  0001 C CNN
-F 3 "~" H 8000 7000 50  0001 C CNN
-	1    8000 7000
-	1    0    0    -1
-$EndComp
 $Comp
 L Device:C C3
@@
 	5950 6150 8950 6150
 Wire Wire Line
-	7200 6050 8950 6050
-Wire Wire Line
 	8000 5950 8950 5950
 Wire Wire Line
@@
 	1    0    0    -1
 $EndComp
-Wire Wire Line
-	13550 8250 13800 8250
 $Comp
 L Device:R R37
@@
 $EndComp
 $Comp
-L Device:C C7
-U 1 1 5EAD43D3
-P 8850 1750
-F 0 "C7" H 8965 1796 50  0000 L CNN
-F 1 "2.2μ" H 8965 1705 50  0000 L CNN
-F 2 "Capacitor_THT:C_Disc_D5.1mm_W3.2mm_P5.00mm" H 8888 1600 50  0001 C CNN
-F 3 "~" H 8850 1750 50  0001 C CNN
-	1    8850 1750
-	1    0    0    -1
-$EndComp
-$Comp
 L power:+5V #PWR024
 U 1 1 5EAC5D04
-P 8850 1400
-F 0 "#PWR024" H 8850 1250 50  0001 C CNN
-F 1 "+5V" H 8865 1573 50  0000 C CNN
-F 2 "" H 8850 1400 50  0001 C CNN
-F 3 "" H 8850 1400 50  0001 C CNN
-	1    8850 1400
-	1    0    0    -1
-$EndComp
-$Comp
-L power:GND #PWR025
-U 1 1 5EAC4E95
-P 8850 2000
-F 0 "#PWR025" H 8850 1750 50  0001 C CNN
-F 1 "GND" H 8855 1827 50  0000 C CNN
-F 2 "" H 8850 2000 50  0001 C CNN
-F 3 "" H 8850 2000 50  0001 C CNN
-	1    8850 2000
-	1    0    0    -1
+P 8650 1500
+F 0 "#PWR024" H 8650 1350 50  0001 C CNN
+F 1 "+5V" V 8650 1700 50  0000 C CNN
+F 2 "" H 8650 1500 50  0001 C CNN
+F 3 "" H 8650 1500 50  0001 C CNN
+	1    8650 1500
+	0    1    1    0
 $EndComp
 Wire Wire Line
@@
 P 8250 1250
 F 0 "R23" H 8320 1296 50  0000 L CNN
-F 1 "680" H 8320 1205 50  0000 L CNN
+F 1 "1k" H 8320 1205 50  0000 L CNN
 F 2 "Resistor_THT:R_Axial_DIN0207_L6.3mm_D2.5mm_P10.16mm_Horizontal" V 8180 1250 50  0001 C CNN
 F 3 "~" H 8250 1250 50  0001 C CNN
 	1    8250 1250
 	1    0    0    -1
-$EndComp
-$Comp
-L Device:D_Zener D2
-U 1 1 5EC1CEB0
-P 8250 1750
-F 0 "D2" V 8204 1829 50  0000 L CNN
-F 1 "1N5231B" V 8295 1829 50  0000 L CNN
-F 2 "Diode_THT:D_DO-34_SOD68_P7.62mm_Horizontal" H 8250 1750 50  0001 C CNN
-F 3 "~" H 8250 1750 50  0001 C CNN
-	1    8250 1750
-	0    1    1    0
 $EndComp
 $Comp
@@
 Wire Wire Line
 	8250 1900 8250 2000
-Wire Wire Line
-	8250 1600 8250 1500
-Wire Wire Line
-	8850 1900 8850 2000
-Wire Wire Line
-	8250 1500 8250 1400
 $Comp
 L power:+12V #PWR020
@@
 	10950 5750 9950 5750
 Wire Wire Line
-	10950 6150 9950 6150
+	10950 6150 10100 6150
 $Comp
 L power:-5V #PWR033
 U 1 1 5F136284
-P 10000 1600
-F 0 "#PWR033" H 10000 1700 50  0001 C CNN
-F 1 "-5V" H 10015 1773 50  0000 C CNN
-F 2 "" H 10000 1600 50  0001 C CNN
-F 3 "" H 10000 1600 50  0001 C CNN
-	1    10000 1600
-	-1   0    0    1
+P 9800 1500
+F 0 "#PWR033" H 9800 1600 50  0001 C CNN
+F 1 "-5V" V 9800 1700 50  0000 C CNN
+F 2 "" H 9800 1500 50  0001 C CNN
+F 3 "" H 9800 1500 50  0001 C CNN
+	1    9800 1500
+	0    1    1    0
 $EndComp
 $Comp
@@
 	-1   0    0    1
 $EndComp
-$Comp
-L Device:D_Zener D3
-U 1 1 5F138EFB
-P 9400 1250
-F 0 "D3" V 9354 1329 50  0000 L CNN
-F 1 "1N5231B" V 9445 1329 50  0000 L CNN
-F 2 "Diode_THT:D_DO-34_SOD68_P7.62mm_Horizontal" H 9400 1250 50  0001 C CNN
-F 3 "~" H 9400 1250 50  0001 C CNN
-	1    9400 1250
-	0    1    1    0
-$EndComp
 Wire Wire Line
 	9400 1000 9400 1100
@@
 P 9400 1750
 F 0 "R26" H 9470 1796 50  0000 L CNN
-F 1 "680" H 9470 1705 50  0000 L CNN
+F 1 "1k" H 9470 1705 50  0000 L CNN
 F 2 "Resistor_THT:R_Axial_DIN0207_L6.3mm_D2.5mm_P10.16mm_Horizontal" V 9330 1750 50  0001 C CNN
 F 3 "~" H 9400 1750 50  0001 C CNN
@@
 	-1   0    0    1
 $EndComp
-$Comp
-L Device:C C9
-U 1 1 5F14CEDC
-P 10000 1250
-F 0 "C9" H 10115 1296 50  0000 L CNN
-F 1 "2.2μ" H 10115 1205 50  0000 L CNN
-F 2 "Capacitor_THT:C_Disc_D5.1mm_W3.2mm_P5.00mm" H 10038 1100 50  0001 C CNN
-F 3 "~" H 10000 1250 50  0001 C CNN
-	1    10000 1250
-	1    0    0    -1
-$EndComp
-$Comp
-L power:GND #PWR032
-U 1 1 5F169E1C
-P 10000 1000
-F 0 "#PWR032" H 10000 750 50  0001 C CNN
-F 1 "GND" H 10005 827 50  0000 C CNN
-F 2 "" H 10000 1000 50  0001 C CNN
-F 3 "" H 10000 1000 50  0001 C CNN
-	1    10000 1000
-	-1   0    0    1
-$EndComp
 Wire Wire Line
 	9400 1900 9400 2000
-Wire Wire Line
-	10000 1100 10000 1000
-Wire Wire Line
-	10000 1400 10000 1500
-Connection ~ 10000 1500
-Wire Wire Line
-	10000 1500 10000 1600
 Wire Wire Line
 	11600 3800 11950 3800
@@
 	1    0    0    -1
 $EndComp
-Wire Wire Line
-	8850 1400 8850 1500
-Wire Wire Line
-	9400 1400 9400 1500
-Wire Wire Line
-	8250 1500 8850 1500
-Connection ~ 8850 1500
-Wire Wire Line
-	8850 1500 8850 1600
-Wire Wire Line
-	9400 1500 10000 1500
-Wire Wire Line
-	9400 1500 9400 1600
 $Comp
 L power:-12V #PWR0102
@@
 Wire Wire Line
 	2600 2600 2600 2650
-Connection ~ 8250 1500
-Connection ~ 9400 1500
 $Comp
 L power:VEE #PWR0109
@@
 	5950 5650 5950 5850
 Connection ~ 5950 5850
+$Comp
+L LM336:LM336 D1
+U 1 1 5F39F7F4
+P 8250 1750
+F 0 "D1" V 8204 1828 50  0000 L CNN
+F 1 "LM336Z-5.0" V 8295 1828 50  0000 L CNN
+F 2 "Package_TO_SOT_THT:TO-92_Inline_Wide" H 8250 1750 50  0001 C CNN
+F 3 "~" H 8250 1750 50  0001 C CNN
+	1    8250 1750
+	0    1    1    0
+$EndComp
+NoConn ~ 8100 1750
+Wire Wire Line
+	8250 1400 8250 1500
+Wire Wire Line
+	8650 1500 8250 1500
+Connection ~ 8250 1500
+Wire Wire Line
+	8250 1500 8250 1600
+Wire Wire Line
+	9400 1400 9400 1500
+Wire Wire Line
+	9800 1500 9400 1500
+Connection ~ 9400 1500
+Wire Wire Line
+	9400 1500 9400 1600
+$Comp
+L LM336:LM336 D2
+U 1 1 5F42C6C2
+P 9400 1250
+F 0 "D2" V 9354 1328 50  0000 L CNN
+F 1 "LM336Z-5.0" V 9445 1328 50  0000 L CNN
+F 2 "Package_TO_SOT_THT:TO-92_Inline_Wide" H 9400 1250 50  0001 C CNN
+F 3 "~" H 9400 1250 50  0001 C CNN
+	1    9400 1250
+	0    1    1    0
+$EndComp
+NoConn ~ 9250 1250
+$Comp
+L Device:C C4
+U 1 1 5E86C6E8
+P 8000 7000
+F 0 "C4" H 8115 7046 50  0000 L CNN
+F 1 "0.1μ" H 8115 6955 50  0000 L CNN
+F 2 "Capacitor_THT:C_Rect_L7.2mm_W5.5mm_P5.00mm_FKS2_FKP2_MKS2_MKP2" H 8038 6850 50  0001 C CNN
+F 3 "~" H 8000 7000 50  0001 C CNN
+	1    8000 7000
+	1    0    0    -1
+$EndComp
+Wire Wire Line
+	8000 6850 8000 6550
+Wire Wire Line
+	13550 8250 13700 8250
+Wire Wire Line
+	7200 6050 8950 6050
+$Comp
+L Connector:TestPoint TP2
+U 1 1 5F66E57C
+P 7900 6550
+F 0 "TP2" V 8095 6622 50  0000 C CNN
+F 1 "VSSI" V 8004 6622 50  0000 C CNN
+F 2 "Connector_PinHeader_2.54mm:PinHeader_1x01_P2.54mm_Vertical" H 8100 6550 50  0001 C CNN
+F 3 "~" H 8100 6550 50  0001 C CNN
+	1    7900 6550
+	0    -1   -1   0
+$EndComp
+Wire Wire Line
+	7900 6550 8000 6550
+Connection ~ 8000 6550
+Wire Wire Line
+	8000 6550 8000 5950
+$Comp
+L Connector:TestPoint TP1
+U 1 1 5F67D91F
+P 7100 6050
+F 0 "TP1" V 7100 6300 50  0000 C CNN
+F 1 "VLFI" V 7204 6122 50  0000 C CNN
+F 2 "Connector_PinHeader_2.54mm:PinHeader_1x01_P2.54mm_Vertical" H 7300 6050 50  0001 C CNN
+F 3 "~" H 7300 6050 50  0001 C CNN
+	1    7100 6050
+	0    -1   -1   0
+$EndComp
+Wire Wire Line
+	7100 6050 7200 6050
+$Comp
+L Connector:TestPoint TP3
+U 1 1 5F68D411
+P 10100 6350
+F 0 "TP3" H 10042 6376 50  0000 R CNN
+F 1 "VTO" H 10042 6467 50  0000 R CNN
+F 2 "Connector_PinHeader_2.54mm:PinHeader_1x01_P2.54mm_Vertical" H 10300 6350 50  0001 C CNN
+F 3 "~" H 10300 6350 50  0001 C CNN
+	1    10100 6350
+	-1   0    0    1
+$EndComp
+Wire Wire Line
+	10100 6350 10100 6150
+Connection ~ 10100 6150
+Wire Wire Line
+	10100 6150 9950 6150
+$Comp
+L Connector:TestPoint TP4
+U 1 1 5F69CD0B
+P 13700 7750
+F 0 "TP4" H 13758 7868 50  0000 L CNN
+F 1 "TRIOUT" H 13758 7777 50  0000 L CNN
+F 2 "Connector_PinHeader_2.54mm:PinHeader_1x01_P2.54mm_Vertical" H 13900 7750 50  0001 C CNN
+F 3 "~" H 13900 7750 50  0001 C CNN
+	1    13700 7750
+	1    0    0    -1
+$EndComp
+Wire Wire Line
+	13700 7750 13700 8250
+Connection ~ 13700 8250
+Wire Wire Line
+	13700 8250 13800 8250
+$Comp
+L power:-12V #PWR0112
+U 1 1 5F728E18
+P 12850 2350
+F 0 "#PWR0112" H 12850 2450 50  0001 C CNN
+F 1 "-12V" V 12850 2600 50  0000 C CNN
+F 2 "" H 12850 2350 50  0001 C CNN
+F 3 "" H 12850 2350 50  0001 C CNN
+	1    12850 2350
+	0    1    1    0
+$EndComp
+$Comp
+L power:+12V #PWR0113
+U 1 1 5F72921D
+P 12850 2250
+F 0 "#PWR0113" H 12850 2100 50  0001 C CNN
+F 1 "+12V" V 12850 2500 50  0000 C CNN
+F 2 "" H 12850 2250 50  0001 C CNN
+F 3 "" H 12850 2250 50  0001 C CNN
+	1    12850 2250
+	0    1    1    0
+$EndComp
+$Comp
+L power:GND #PWR0114
+U 1 1 5F7299E2
+P 12850 2450
+F 0 "#PWR0114" H 12850 2200 50  0001 C CNN
+F 1 "GND" V 12850 2200 50  0000 C CNN
+F 2 "" H 12850 2450 50  0001 C CNN
+F 3 "" H 12850 2450 50  0001 C CNN
+	1    12850 2450
+	0    -1   -1   0
+$EndComp
+$Comp
+L Connector_Generic:Conn_01x03 J8
+U 1 1 5F7C29A7
+P 12550 2350
+F 0 "J8" H 12468 2025 50  0000 C CNN
+F 1 "EXT_POW" H 12468 2116 50  0000 C CNN
+F 2 "Connector_PinHeader_2.54mm:PinHeader_1x03_P2.54mm_Vertical" H 12550 2350 50  0001 C CNN
+F 3 "~" H 12550 2350 50  0001 C CNN
+	1    12550 2350
+	-1   0    0    1
+$EndComp
+Wire Wire Line
+	12850 2250 12750 2250
+Wire Wire Line
+	12750 2350 12850 2350
+Wire Wire Line
+	12850 2450 12750 2450
 $EndSCHEMATC
