File: pcb_main/3340VCO_pcb_main.kicad_pcb (KiCad board)
At the start: 2 copper layers, 60 x 109.5 mm, 77 parts, among them J1 MJ-352, J2 MJ-352, J3 MJ-352, J4 POWER_IN, J5 MJ-352, J6 MJ-352, J7 MJ-352, U1 NJM074, U2 NJM074, U3 V3340M

Commit message: replace reference Diode: 1N5231B to LM336Z-5.0, update schematic and pcb
Parts:
- removed C7, C9: 2.2μ, Capacitor_THT:C_Disc_D5.1mm_W3.2mm_P5.00mm
- removed D3: 1N5231B, Diode_THT:D_DO-34_SOD68_P7.62mm_Horizontal
- added D1: LM336Z-5.0, Package_TO_SOT_THT:TO-92_Inline_Wide, F.Cu at (66.4, 91.3)
- added J8: EXT_POW, Connector_PinHeader_2.54mm:PinHeader_1x03_P2.54mm_Vertical, F.Cu at (58.6, 123.7)
- added TP1: VLFI, Connector_PinHeader_2.54mm:PinHeader_1x01_P2.54mm_Vertical, F.Cu at (85.5, 89.3)
- added TP2: VSSI, Connector_PinHeader_2.54mm:PinHeader_1x01_P2.54mm_Vertical, F.Cu at (92.9, 100.8)
- added TP3: VTO, Connector_PinHeader_2.54mm:PinHeader_1x01_P2.54mm_Vertical, F.Cu at (94.9, 104.6)
- added TP4: TRIOUT, Connector_PinHeader_2.54mm:PinHeader_1x01_P2.54mm_Vertical, F.Cu at (92.7, 141.3)
- C4: value 10n -> 0.1μ; footprint C_addition:C_Rect_L4.0mm_W2.5mm_P2.50mm -> Capacitor_THT:C_Rect_L7.2mm_W5.5mm_P5.00mm_FKS2_FKP2_MKS2_MKP2
- D2: value 1N5231B -> LM336Z-5.0; footprint Diode_THT:D_DO-34_SOD68_P7.62mm_Horizontal -> Package_TO_SOT_THT:TO-92_Inline_Wide
- R23, R26: value 680 -> 1k
- moved D2 48.9 mm to (57.0, 141.8)
- moved C4 2.61 mm to (92.9, 97.2)
Connections:
- D2 pad 1: +5V -> (no net)
Routing:
- net Net-(R18-Pad2): track 12.5 -> 19.0 mm
- net Net-(J7-PadT): track 13.3 -> 18.3 mm
- net Net-(C4-Pad1): track 10.7 -> 14.4 mm
- net Net-(R29-Pad2): track 9.19 -> 12.7 mm
- net -5V: track 63.1 -> 60.2 mm
- net +5V: track 79.0 -> 80.3 mm

Commit message: migrate to KiCAD 6.0
Connections:
- D1 pad 1: (no net) -> unconnected-(D1-Pad1)
- D2 pad 1: (no net) -> unconnected-(D2-Pad1)
- J1 pad TN: (no net) -> unconnected-(J1-PadTN)
- J2 pad TN: (no net) -> unconnected-(J2-PadTN)
- J3 pad TN: (no net) -> unconnected-(J3-PadTN)
- J4 pad 11: (no net) -> unconnected-(J4-Pad11)
- J4 pad 12: (no net) -> unconnected-(J4-Pad12)
- J4 pad 13: (no net) -> unconnected-(J4-Pad13)
- J4 pad 14: (no net) -> unconnected-(J4-Pad14)
- J4 pad 15: (no net) -> unconnected-(J4-Pad15)
- J4 pad 16: (no net) -> unconnected-(J4-Pad16)
- J5 pad TN: (no net) -> unconnected-(J5-PadTN)
- J6 pad TN: (no net) -> unconnected-(J6-PadTN)
- J7 pad TN: (no net) -> unconnected-(J7-PadTN)
Other:
- net class Bold removed
- net class Default removed
